File: pcb/pcb.kicad_pcb (KiCad board)
At the start: 2 copper layers, 117 x 96 mm, 50 parts, among them J1 BATT, J2 BATT, SW1 SW_SPST, SW10 SW_SPST, SW11 SW_SPST, SW12 SW_SPST, SW13 SW_SPST, SW14 SW_SPST, SW15 SW_SPST, SW16 SW_SPST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

Commit message: V1.2: fix missing traces on right half
Routing:
- net Net-(D10-A): track 20.7 -> 22.4 mm
- net Net-(D18-A): track 20.8 -> 22.4 mm
Other:
- board text added: "Ergonaut One S v1.2 by Ladniy"
- board text removed: "Ergonaut One S v1.1 by Ladniy"
